File: hardware/gambos-pcb/MCU.kicad_sch (KiCad schematic)
At the start: 85 parts, among them J10 Conn_01x03_Pin, J11 Conn_01x03_Pin, J12 Conn_01x03_Pin, J13 Conn_01x03_Pin, J14 Conn_01x06_Pin, J15 Conn_01x01_Pin, J16 Conn_01x01_Pin, J17 Conn_01x01_Pin, J18 Conn_01x01_Pin, J19 Conn_01x01_Pin, J2 Conn_01x04_Pin, J20 Conn_01x01_Pin, J21 Conn_01x01_Pin, J22 Conn_01x01_Pin, J5 Conn_01x03_Pin, J7 Conn_01x03_Pin, J9 Conn_01x03_Pin, SW1 SW_Push, SW3 SW_Push, SW4 SW_SPDT, U1 BME280, U3 LIS2MDLTR, U5 W25Q128JVSIQ, U6 LSM6DSVTR, U7 STM32F446RET6, U8 MCP1825S, U9 SN74AHCT244N, Y2 TSX-3225_26MHZ

Commit message: Finished version before checks from hw engineers
Parts:
- removed C10, C11, C12, C13, C15, C16, C17, C18, C19, C28, C3: 100n, Capacitor_SMD:C_0603_1608Metric, symbol Device:C
- removed C20: 10u, Capacitor_SMD:C_0603_1608Metric, symbol Device:C
- removed C21: 4.7u, Capacitor_SMD:C_0603_1608Metric, symbol Device:C
- removed C22: 1u, Capacitor_SMD:C_0603_1608Metric, symbol Device:C
- removed C23, C24, C25, C26, C27: 470u, Capacitor_THT:C_Radial_D4.0mm_H5.0mm_P1.50mm, symbol Device:C
- removed C29, C30: 10p, Capacitor_SMD:C_0603_1608Metric, symbol Device:C
- removed C31: 220n, Capacitor_SMD:C_0603_1608Metric, symbol Device:C
- removed D1: LED0, LED_SMD:LED_0603_1608Metric, symbol Device:LED
- removed D2: LED1, LED_SMD:LED_0603_1608Metric, symbol Device:LED
- removed D3: LED2, LED_SMD:LED_0603_1608Metric, symbol Device:LED
- removed D4: LED3, LED_SMD:LED_0603_1608Metric, symbol Device:LED
- removed J10, J11, J12, J13, J5, J7, J9: Conn_01x03_Pin, Connector_PinHeader_1.00mm:PinHeader_1x03_P1.00mm_Vertical, symbol Connector:Conn_01x03_Pin
- removed J14: Conn_01x06_Pin, Connector_PinHeader_1.00mm:PinHeader_1x06_P1.00mm_Vertical, symbol Connector:Conn_01x06_Pin
- removed J15, J16, J17, J18, J19, J20, J21, J22: Conn_01x01_Pin, Connector_Wire:SolderWire-0.1sqmm_1x01_D0.4mm_OD1mm, symbol Connector:Conn_01x01_Pin
- removed J2: Conn_01x04_Pin, Connector_PinHeader_1.00mm:PinHeader_1x04_P1.00mm_Vertical, symbol Connector:Conn_01x04_Pin
- removed R1: 10k, Resistor_SMD:R_0402_1005Metric, symbol Device:R
- removed R10: 100k, Resistor_SMD:R_0402_1005Metric, symbol Device:R
- removed R2: 10K, symbol Device:R
- removed R3, R4: 4k2, Resistor_SMD:R_0402_1005Metric, symbol Device:R
- removed R5: 1k5, Resistor_SMD:R_0402_1005Metric, symbol Device:R
- removed R6, R8, R9: 130R, Resistor_SMD:R_0402_1005Metric, symbol Device:R
- removed R7: 47k, Resistor_SMD:R_0402_1005Metric, symbol Device:R
- removed SW1, SW3: SW_Push, Button_Switch_SMD:SW_Push_1P1T_NO_E-Switch_TL3301NxxxxxG, symbol Switch:SW_Push
- removed SW4: SW_SPDT, symbol Switch:SW_SPDT
- removed TP10, TP3, TP4, TP5, TP6, TP7, TP8, TP9: TestPoint, TestPoint:TestPoint_Pad_D1.0mm, symbol Connector:TestPoint
- removed U1: BME280, gambos-pcb:PSON65P250X250X100-8N, symbol gambos-symbols:BME280
- removed U3: LIS2MDLTR, gambos-pcb:PQFN50P200X200X70-12N, symbol gambos-symbols:LIS2MDLTR
- removed U5: W25Q128JVSIQ, gambos-pcb:SOIC127P790X216-8N, symbol gambos-symbols:W25Q128JVSIQ
- removed U6: LSM6DSVTR, gambos-pcb:LGA14-L_2P59X3P1X0P5_STM-L, symbol gambos-symbols:LSM6DSVTR
- removed U7: STM32F446RET6, gambos-pcb:QFP50P1200X1200X160-64N, symbol gambos-symbols:STM32F446RET6
- removed U8: MCP1825S, Package_TO_SOT_SMD:SOT-223-3_TabPin2, symbol Regulator_Linear:MCP1825S
- removed U9: SN74AHCT244N, gambos-pcb:SN74AHCT244N, symbol gambos-symbols:SN74AHCT244N
- removed Y2: TSX-3225_26MHZ, gambos-pcb:QFP50P1200X1200X160-64N, symbol gambos-symbols:TSX-3225_26.0000MF09Z-AC0
- added C33: 100n, Capacitor_SMD:C_0603_1608Metric, symbol Device:C
- added TVS2, TVS3, TVS4, TVS6, TVS7: DESD5V0U1BA-7, gambos-pcb:DESD5V0U1BA-7, symbol gambos-symbols:DESD5V0U1BA-7
- added U1: NRF24L01_Breakout, RF_Module:nRF24L01_Breakout, symbol RF:NRF24L01_Breakout
- added U2: D1213A-04S-7, gambos-pcb:D1213A-04S-7, symbol gambos-symbols:D1213A-04S-7
Connections:
- net +3V3: now also C33.1, U1.2 (VCC), U2.5 (VP)
- net GND: now also C33.2, TVS2.1, TVS3.1, TVS4.1, TVS6.1, TVS7.1, U1.1 (GND), U2.2 (VN)
- net IRQ_SLD: now also U1.8 (IRQ)
- net NRF24_CE_SLD: now also U1.3 (CE)
- net NRF24_CS_SLD: now also U1.4 (~{CSN})
- net NRST: now also TVS2.2
- net SWCLK: now also U2.3 (CH2)
- net SWDIO: now also U2.1 (CH1)
- net SWO: now also TVS3.2
- net UART4_RX: now also U2.4 (CH3)
- net UART4_TX: now also U2.6 (CH4)
- new net SPI1.MISO_1: U1.7 (MISO)
- new net SPI1.MOSI_1: U1.6 (MOSI)
- new net SPI1.SCK_1: U1.5 (SCK)
- new net TVS_BOOT0: TVS6.2
- new net TVS_NRST: TVS7.2
- new net TVS_USER_BTN: TVS4.2
- no-connect marks 33 -> 0
Other:
- added sheet Microcontroller (microcontroller.kicad_sch)
- added sheet Power and ESC (power_and_esc.kicad_sch)
- added sheet Sensors and flash (sensors_and_flash.kicad_sch)
- added sheet Servos and connectors (servo_connectors.kicad_sch)
- note added: "ESD protection"
- note added: "Mounting holes"
- note added: "nRF module solder points"
- note removed: "2*(9-4)=10pF"
- note removed: "5*RC = 23.5ms"
- note removed: "BEC"
- note removed: "Boot and Reset"
- note removed: "Crystal oscillator"
- note removed: "External flash"
- note removed: "Gyro and accelerometer"
- note removed: "Logic level shifter"
- note removed: "Low ESR, X7R or X5R Ceramic"
- note removed: "Magnetometer"
- note removed: "Microcontroller"
- note removed: "NRF module solder points, mounting holes and test points"
- note removed: "Power supply"
- note removed: "Pressure and humidity"
- note removed: "R=(3.3-2)/0.01=130 Ohm"
- note removed: "SWD and UART"
- note removed: "Servo-motor headers and capacitors"
- note removed: "User button and LED"
- moved on the sheet: C1, C2, C4, C5, C6, C7, C8, C9, FB1, H1, H2, H3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
