File: hardware/gambos-pcb/gambos-pcb.kicad_sch (KiCad schematic)
At the start: 0 parts

Commit message: Finished version before checks from hw engineers
Other:
- note added: "SWD with UART"
- note removed: "SWD with power and UART"
Changed lines of the file:
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@@
 		)
 	)
-	(text "SWD with power\nand UART\n"
+	(text "SWD with UART\n"
 		(exclude_from_sim no)
-		(at 119.38 63.5 0)
+		(at 120.396 63.5 0)
 		(effects
 			(font
@@
 		)
 		(stroke
-			(width 0)
-			(type default)
-		)
-	)
-	(bus
-		(pts
-			(xy 121.92 67.31) (xy 121.92 77.47)
-		)
-		(stroke
